Commit message: Gazebo: First /cmd_vel responsive version

File: pet_mk_iv_description/urdf/pet_mk_iv.urdf.xacro (robot description, xacro)
@@ -62,7 +62,18 @@
       <origin xyz="0.0 0 0.0" rpy=" 0 0 0"/>
       <inertia
-          ixx="0.1" ixy="0" ixz="0"
-          iyy="0.1" iyz="0"
-          izz="0.1"/>
+          ixx="0.007"
+          ixy="-2.0E-08"
+          ixz="0.000014"
+          iyy="0.0007"
+          iyz="4.6E-09"
+          izz="0.0011"/>
+<!-- froom Tianbot-Mini
+          ixx="6.9553958488565E-04"
+          ixy="-1.99945013904458E-08"
+          ixz="1.43938674591944E-05"
+          iyy="7.30544716315262E-04"
+          iyz="4.63385578966379E-09"
+          izz="0.0011040368246549"
+-->
     </inertial>
   </link>
@@ -93,4 +104,22 @@
       <material name="green"/>
     </visual>
+    <xacro:property name="body_thicknes_upper_deck" value="0.020"/>
+    <xacro:property name="body_hight_upper_deck" value="0.060"/>
+    <xacro:property name="body_thicknes_lower_deck" value="0.030"/>
+    <xacro:property name="body_hight_lower_deck" value="${body_thicknes_lower_deck/2}"/>
+    <collision name='body_upper_deck_collision'>
+      <origin xyz="0 0 ${body_hight_upper_deck}" rpy=" 0 0 0"/>
+      <geometry>
+        <box size= "${body_length} ${body_width} ${body_thicknes_upper_deck}"/>
+      </geometry>
+      <material name="green"/>
+    </collision>
+    <collision name='body_lower_deck_collision'>
+      <origin xyz="0 0 ${body_hight_lower_deck}" rpy=" 0 0 0"/>
+      <geometry>
+        <box size= "${body_length} ${body_width} ${body_thicknes_lower_deck}"/>
+      </geometry>
+      <material name="green"/>
+    </collision>
 <!--
     <collision name='main_body_collision'>
@@ -102,5 +131,5 @@
 -->
     <collision name='main_body_grip_collision'>
-      <origin xyz="0 0 ${body_hight/2}" rpy=" 0 0 0"/>
+      <origin xyz="0 0 ${body_hight/2+0.055}" rpy=" 0 0 0"/>
       <geometry>
         <box size= "0.015 0.135 0.070"/>  <!-- Cube of Robot Grip -->

File: pet_mk_iv_description/urdf/pet_mk_iv_gazebo.urdf.xacro (robot description, xacro)
@@ -46,6 +46,6 @@
       <alwaysOn>true</alwaysOn>      <!-- ??? Is this valid for this Gazebo plugin??? -->
       <updateRate>10</updateRate>    <!-- Plugin update rate in Hz -->
-      <leftJoint>left_front_wheel_joint</leftJoint>    <!-- Name of left joint, defaults to `left_joint` -->
-      <rightJoint>right_front_wheel_joint</rightJoint> <!-- Name of right joint, defaults to `right_joint` -->
+      <leftJoint>front_left_wheel_joint</leftJoint>    <!-- Name of left joint, defaults to `left_joint` -->
+      <rightJoint>front_right_wheel_joint</rightJoint> <!-- Name of right joint, defaults to `right_joint` -->
       <wheelSeparation>0.54</wheelSeparation>    <!-- The distance from the center of one wheel to the other, in meters, defaults to 0.34 m -->
       <wheelDiameter>0.26</wheelDiameter>        <!-- Diameter of the wheels, in meters, defaults to 0.15 m -->

File: pet_mk_iv_description/urdf/wheel.urdf.xacro (robot description, xacro)
@@ -48,10 +48,29 @@
       <inertial>
         <origin xyz="0 0 0" rpy="0 1.5707 1.5707"/>
-        <mass value="5"/>
+        <mass value="0.01" />
         <inertia
-          ixx=".1" ixy="0.0" ixz="0.0"
-          iyy=".1" iyz="0.0"
-          izz=".1"/>
+          ixx="2.40384090487514E-05"
+          ixy="9.21491839222917E-12"
+          ixz="1.16650464760408E-11"
+          iyy="4.21578178329362E-05"
+          iyz="2.56744598636029E-11"
+          izz="2.40355678533584E-05"/>
       </inertial>
+<!-- from Tianbot-Mini: Left wheel
+          ixx="2.40384090487514E-05"
+          ixy="9.21491839222917E-12"
+          ixz="1.16650464760408E-11"
+          iyy="4.21578178329362E-05"
+          iyz="2.56744598636029E-11"
+          izz="2.40355678533584E-05"
+-->
+<!-- from Tianbot-Mini: Right wheel
+          ixx="2.40403731664504E-05"
+          ixy="1.93558318570861E-11"
+          ixz="-1.9701375781678E-11"
+          iyy="4.21599888385316E-05"
+          iyz="3.15208827782047E-12"
+          izz="2.4035775665164E-05"
+-->
     </link>
     <joint type="continuous" name="${wheel_prefix}_wheel_joint">

Commit message: Minor fixes... :-)

File: pet_mk_iv_description/urdf/pet_mk_iv.urdf.xacro (robot description, xacro)
@@ -19,5 +19,5 @@
 -->
 <robot name="Pet Mk.IV" xmlns:xacro="http://www.ros.org/wiki/xacro">
-  <xacro:include filename="$(find pet_mk_iv_description)/urdf/materials.xacro"/>
+  <xacro:include filename="$(find pet_mk_iv_description)/urdf/materials.xacro"/>    <!-- Import Rviz colors -->
   <xacro:include filename="$(find pet_mk_iv_description)/urdf/pet_mk_iv_gazebo.urdf.xacro" />
   <xacro:include filename="$(find pet_mk_iv_description)/urdf/sensor_hc_sr04_sonarRange.urdf.xacro"/>
@@ -28,7 +28,7 @@
   <xacro:include filename="$(find pet_mk_iv_description)/urdf/wheel.urdf.xacro"/>
   <xacro:include filename="$(find pet_mk_iv_description)/urdf/visual_raspberryPi3B_sbc.urdf.xacro"/>
-  <xacro:property name="robot_weight"       value="0.9"/>    <!-- unit kg  -->
+  <xacro:property name="robot_weight"    value="0.9"/>    <!-- unit kg  -->
   <xacro:property name="sonar_center_height" value="0.060"/>   <!-- unit m  -->
-  <xacro:property name="PI" value="3.14159265359"/>   <!-- unit n/a  -->
+  <xacro:property name="PI"              value="3.14159265359"/>   <!-- unit n/a  -->
   <xacro:property name="chassis_height"  value="0.020"/>   <!-- unit m  -->
 <!--
@@ -112,5 +112,5 @@
     <visual name='Pet_Mk_IV_body_visual'>
       <origin xyz="0 0 0" rpy="${PI/2} 0 ${PI}"/>
-      <geometry>'
+      <geometry>
 <!--
       ???????????????????????????????????????????????????????????????????????????

Commit message: PET-28_Updated URDF  with grip&bracket

File: pet_mk_iv_description/urdf/pet_mk_iv.urdf.xacro (robot description, xacro)
@@ -130,10 +130,43 @@
       <material name='brown'/>   <!-- Color in RViz -->
     </visual>
-    <visual name='Pet_Mk_IV_body_grip_link_visual'>
-      <origin xyz="0 0 ${body_height/2+0.055}" rpy=" 0 0 0"/>
-      <geometry>
-        <box size= "0.015 0.135 0.070"/>
-      </geometry>
-      <material name="green"/>
+    <visual name='Pet_Mk_IV_body_grip_rightBracket_link_visual'>
+      <origin xyz="0 ${+0.132/2} ${body_height-0.004-0.002+0.070/2}" rpy=" 0 0 0"/>
+      <geometry>
+        <box size= "0.015 0.002 0.070"/>    <!-- Right vertical bracket holding grip -->
+      </geometry>
+      <material name="blue"/>
+    </visual>
+    <visual name='Pet_Mk_IV_body_grip_leftBracket_link_visual'>
+      <origin xyz="0 ${-0.132/2} ${body_height-0.004-0.002+0.070/2}" rpy=" 0 0 0"/>
+      <geometry>
+        <box size= "0.015 0.002 0.070"/>    <!-- Left vertical bracket holding grip -->
+      </geometry>
+      <material name="blue"/>
+    </visual>
+    <visual name='Pet_Mk_IV_body_grip_bracket_link_visual'>
+      <origin xyz="0 0 ${body_height-0.004-0.002}" rpy=" 0 0 0"/>
+      <geometry>
+        <box size= "0.015 0.132 0.002"/>    <!-- Horizontal bracket -->
+      </geometry>
+      <material name="blue"/>
+    </visual>
+    <visual name='Pet_Mk_IV_body_grip_horisontal_link_visual'>
+      <origin xyz="0 0 ${body_height+0.056}" rpy=" 0 0 0"/>
+      <geometry>
+        <box size= "0.009 0.132 0.015"/>    <!-- Horizontal beam/grip -->
+      </geometry>
+      <material name="brown"/>
+    </visual>
+    <visual name='Pet_Mk_IV_body_lightBeacon_link_visual'>
+      <origin xyz="0 ${body_width/2} ${body_height+0.072}" rpy=" 0 0 0"/>
+      <geometry>
+        <cylinder radius="0.006" length="0.018"/>    <!-- LightBeacon -->
+      </geometry>
+      <material name="LED material">
+        <ambient>0 0 0 1</ambient>
+        <diffuse>0 0 0 1</diffuse>
+        <specular>0 0 0 0</specular>
+        <emissive>0 1 0 1</emissive>
+      </material>
     </visual>
     <collision name='Pet_Mk_IV_body_grip_collision'>

Commit message: PET-28_New URDF.xacro for LCD1602-display

File: pet_mk_iv_description/urdf/pet_mk_iv.urdf.xacro (robot description, xacro)
@@ -28,8 +28,9 @@
   <xacro:include filename="$(find pet_mk_iv_description)/urdf/wheel.urdf.xacro"/>
   <xacro:include filename="$(find pet_mk_iv_description)/urdf/visual_raspberryPi3B_sbc.urdf.xacro"/>
-  <xacro:property name="robot_weight"       value="0.9"/>    <!-- unit kg  -->
-  <xacro:property name="sonar_center_height" value="0.060"/>   <!-- unit m  -->
-  <xacro:property name="PI" value="3.14159265359"/>   <!-- unit n/a  -->
-  <xacro:property name="chassis_height"  value="0.020"/>   <!-- unit m  -->
+  <xacro:include filename="$(find pet_mk_iv_description)/urdf/visual_LCD1602.urdf.xacro"/>
+  <xacro:property name="robot_weight"        value="0.9"/>    <!-- unit kg  -->
+  <xacro:property name="sonar_center_height" value="0.060"/>  <!-- unit m  -->
+  <xacro:property name="PI" value="3.14159265359"/>           <!-- unit n/a  -->
+  <xacro:property name="chassis_height"  value="0.020"/>      <!-- unit m  -->
 <!--
   Future implementation... Not used yet!
@@ -238,3 +239,9 @@
                 origin_xyz="0.005 -0.005 0.095"
                 origin_rpy="0 0 ${PI/2}"/>
+  <!--
+    Call COSMETIC BODY PART MACRO's: Creates link + joint vs."base_link"
+  -->
+  <xacro:visual_LCD1602 display_name="display_LCD1602"
+                origin_xyz="-0.055 -0.009 0.095"
+                origin_rpy="0 0 0"/>
 </robot>
